Commit message: sensor urdf models added, gmapping launch file still testing

File: turtlebot_model/robots/kobuki_hexagons_d435.urdf.xacro (robot description, xacro)
@@ -3,5 +3,6 @@
     - Base      : kobuki
     - Stacks    : hexagons
-    - 3d Sensor : kinect
+    - 3d Sensor : d435
+    - 3d Sensor : Velodyne VLP-16
 -->
 <robot name="turtlebot" xmlns:xacro="http://ros.org/wiki/xacro">
@@ -10,6 +11,15 @@
   <xacro:include filename="$(find turtlebot_mqp)/turtlebot_model/urdf/stacks/hexagons.urdf.xacro"/>
   <xacro:include filename="$(find turtlebot_mqp)/turtlebot_model/urdf/sensors/_d435.urdf.xacro"/>
+  <xacro:include filename="$(find turtlebot_mqp)/turtlebot_model/urdf/sensors/VLP-16.urdf.xacro"/>
   <xacro:kobuki/>
   <xacro:stack_hexagons parent="base_link"/>
-  <xacro:sensor_d435 parent="base_link"/>
+  <!-- origin, top surface of top plate:0.3972, top pole height: 0.0936-->
+  <!-- d435 height: .025, total:0.0497-->
+  <xacro:sensor_d435 name="d435" parent="base_link">
+    <origin xyz="0 0 0.3972" rpy="0 0 0" />
+  </xacro:sensor_d435>
+  <!-- VLP height: 0.0717-->
+  <xacro:VLP-16 name="VLP-16" parent="base_link">
+    <origin xyz="-0.015 0 0.4908" rpy="0 0 0" />
+  </xacro:VLP-16>
 </robot>

File: turtlebot_model/urdf/sensors/_d435.urdf.xacro (robot description, xacro)
@@ -9,5 +9,6 @@
   <!-- Includes -->
   <xacro:include filename="$(find realsense2_description)/urdf/_materials.urdf.xacro" />
-  <xacro:macro name="sensor_d435" params="parent *origin name:=camera use_nominal_extrinsics:=false">
+  <xacro:include filename="$(find turtlebot_description)/urdf/common_properties.urdf.xacro"/>
+  <xacro:macro name="sensor_d435" params="parent *origin name:=camera use_nominal_extrinsics:=true">
     <xacro:property name="M_PI" value="3.1415926535897931" />
     <!-- The following values are approximate, and the camera node
@@ -62,5 +63,5 @@
     </link>
     <!-- Use the nominal extrinsics between camera frames if the calibrated extrinsics aren't being published. e.g. running the device in simulation  -->
-    <xacro:if value="$(arg use_nominal_extrinsics)">
+    <xacro:if value="${use_nominal_extrinsics}"> <!-- $(arg use_nominal_extrinsics) -->
       <!-- camera depth joints and links -->
       <joint name="${name}_depth_joint" type="fixed">

File: turtlebot_model/urdf/stacks/hexagons.urdf.xacro (robot description, xacro)
@@ -193,6 +193,6 @@
     <xacro:stack_top_pole parent="${parent}" number="2" x_loc="-0.0381" y_loc= "0.1505" z_loc="0.2920"/>
     <xacro:stack_top_pole parent="${parent}" number="3" x_loc="-0.0381" y_loc="-0.1505" z_loc="0.2920"/>
-    <xacro:stack_3d_sensor_pole parent="${parent}" number="0" x_loc="-0.1024" y_loc= "0.098" z_loc="0.2372"/>
-    <xacro:stack_3d_sensor_pole parent="${parent}" number="1" x_loc="-0.1024" y_loc="-0.098" z_loc="0.2372"/>
+    <xacro:stack_3d_sensor_pole parent="${parent}" number="0" x_loc="0.0000" y_loc= "0.1505" z_loc="0.4440"/> <!-- x=-0.1024 y=0.098 -->
+    <xacro:stack_3d_sensor_pole parent="${parent}" number="1" x_loc="0.0000" y_loc="-0.1505" z_loc="0.4440"/> <!-- x=-0.1024 y=-0.098 -->
     <joint name="plate_top_joint" type="fixed">
       <origin xyz="-0.01364 0.0  0.3966" rpy="0 0 0"/>
